Commit message: Convert T-shape geometry from cylinders to rectangular boxes

File: projects/3d/gazebo/joint1/urdf/t_shape.urdf (robot description, URDF)
Before this commit: robot t_shape, 3 links, 2 joints
Links:
- link crossbar: geometry collision box size=0.8 0.1 0.1; visual box size=0.8 0.1 0.1
- link stem: geometry collision box size=0.1 0.1 1.0; visual box size=0.1 0.1 1.0

Commit message: Add hanging green-gradient arm on revolute joint via embedded connector pin

File: projects/3d/gazebo/joint1/urdf/t_shape.urdf (robot description, URDF)
Before this commit: robot t_shape, 3 links, 2 joints
Links:
- added link arm, mass 0.5; collision box size=0.1 0.1 0.5; visual box size=0.1 0.1 0.5
- added link connector, mass 0.15; collision cylinder length=0.20 radius=0.02; visual cylinder length=0.20 radius=0.02
Joints:
- added joint connector_to_arm: type revolute, parent crossbar, child arm, origin xyz=0.35 0.11 0 rpy=0 0 0, axis 0 1 0, limit lower=-3.14159 upper=3.14159 effort=100.0 velocity=10.0
- added joint crossbar_to_connector: type fixed, parent crossbar, child connector, origin xyz=0.35 0 0 rpy=0 0 0

Commit message: Rebuild T-shape from Blender STL meshes; fix crossbar position to form proper T

File: projects/3d/gazebo/joint1/urdf/t_shape.urdf (robot description, URDF)
Before this commit: robot t_shape, 5 links, 4 joints
Links:
- link arm: geometry collision mesh filename=file:///home/ben/dev/design-engine/projects/3d/gazebo/joint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 scale=0.1 0.1 0.1; visual mesh filename=file:///home/ben/dev/design-engine/projects/3d/gazebo/joint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 scale=0.1 0.1 0.1
- link connector: geometry collision mesh filename=file:///home/ben/dev/design-engine/projects/3d/gazebo/joint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 scale=0.1 0.1 0.1; visual mesh filename=file:///home/ben/dev/design-engine/projects/3d/gazebo/joint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 scale=0.1 0.1 0.1
- link crossbar: geometry collision mesh filename=file:///home/ben/dev/design-engine/projects/3d/gazebo/joint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 scale=0.1 0.1 0.1; visual mesh filename=file:///home/ben/dev/design-engine/projects/3d/gazebo/joint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 scale=0.1 0.1 0.1
- link stem: geometry collision mesh filename=file:///home/ben/dev/design-engine/projects/3d/gazebo/joint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 scale=0.1 0.1 0.1; visual mesh filename=file:///home/ben/dev/design-engine/projects/3d/gazebo/joint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 scale=0.1 0.1 0.1
Joints:
- joint connector_to_arm: axis 0 1 0 -> 1 0 0; origin xyz=0.35 0.11 0 rpy=0 0 0 -> xyz=0.22 0.40 0.0056 rpy=0 0 0
- joint crossbar_to_connector: origin xyz=0.35 0 0 rpy=0 0 0 -> xyz=0.15 0.40 0.0056 rpy=0 0 0
