Commit message: g1-sim: 123

File: projects/3d/gazebo/urdf-humanoid/urdf/g1_torso.urdf (robot description, URDF)
Before this commit: robot g1_29dof, 30 links, 29 joints
Links:
- link head_link: geometry collision box size=0.125 0.14 0.185; visual mesh filename=file:///home/ben/dev/design-engine/projects/3d/gazebo/urdf-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
- link left_elbow_link: geometry collision cylinder length=0.11 radius=0.03; visual mesh filename=file:///home/ben/dev/design-engine/projects/3d/gazebo/urdf-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
- link left_rubber_hand: geometry collision box size=0.115 0.058 0.095; visual mesh filename=file:///home/ben/dev/design-engine/projects/3d/gazebo/urdf-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
- link left_shoulder_yaw_link: geometry collision cylinder length=0.115 radius=0.03; visual mesh filename=file:///home/ben/dev/design-engine/projects/3d/gazebo/urdf-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
- link left_wrist_pitch_link: geometry collision cylinder length=0.085 radius=0.026; visual mesh filename=file:///home/ben/dev/design-engine/projects/3d/gazebo/urdf-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
- link left_wrist_roll_link: geometry collision sphere radius=0.026; visual mesh filename=file:///home/ben/dev/design-engine/projects/3d/gazebo/urdf-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
- link left_wrist_yaw_link: geometry collision sphere radius=0.026; visual mesh filename=file:///home/ben/dev/design-engine/projects/3d/gazebo/urdf-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
- link right_elbow_link: geometry collision cylinder length=0.11 radius=0.03; visual mesh filename=file:///home/ben/dev/design-engine/projects/3d/gazebo/urdf-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
- link right_rubber_hand: geometry collision box size=0.115 0.058 0.095; visual mesh filename=file:///home/ben/dev/design-engine/projects/3d/gazebo/urdf-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
- link right_shoulder_yaw_link: geometry collision cylinder length=0.115 radius=0.03; visual mesh filename=file:///home/ben/dev/design-engine/projects/3d/gazebo/urdf-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
- link right_wrist_pitch_link: geometry collision cylinder length=0.085 radius=0.026; visual mesh filename=file:///home/ben/dev/design-engine/projects/3d/gazebo/urdf-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
- link right_wrist_roll_link: geometry collision sphere radius=0.026; visual mesh filename=file:///home/ben/dev/design-engine/projects/3d/gazebo/urdf-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
- link right_wrist_yaw_link: geometry collision sphere radius=0.026; visual mesh filename=file:///home/ben/dev/design-engine/projects/3d/gazebo/urdf-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
- link torso_link: geometry collision box size=0.135 0.195 0.295; visual mesh filename=file:///home/ben/dev/design-engine/projects/3d/gazebo/urdf-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
