Commit message: arm-rig: passive revolute shoulder + upper arm
Hangs an upper arm off the right end (-Y) of the crossbar.

- upper_arm: 0.07 x 0.07 x 0.75 m, length derived as stem_height/2 so it
  tracks the stem if that is rescaled
- shoulder_joint: revolute about X, swinging in the Y-Z plane, +/-pi
- deliberately passive - damping 0.2 / friction 0.1, no transmission and
  no controller, so it falls and swings under gravity like the g1 torso
  rig does
- link frame at the pivot with geometry offset -length/2, so the arm
  hangs below the joint; tip rests 0.75 m clear of the ground

File: projects/3d/gazebo/URDF-Humanoid-Arm/urdf/rig.urdf.xacro (robot description, xacro)
@@ -1,18 +1,25 @@
 <?xml version="1.0"?>
 <!--
-  Stage 2: a vertical stem welded to the world, with a horizontal crossbar
-  sitting on top of it. A plain "T".
+  Stage 3: vertical stem welded to the world, horizontal crossbar on top,
+  and an upper arm hanging from the RIGHT end of the crossbar on a free
+  revolute joint.
   Convention used throughout: every link's own frame sits at the point where
   it attaches to its parent, and the geometry is offset from there. That
   keeps the joint origins trivial and lets the rig rescale cleanly when the
   parameters change.
-    stem     - frame at ground level, box pushed up by stem_height/2 so it
-               stands ON the ground instead of being half buried. Its top
-               face therefore lands at exactly z = stem_height.
-    crossbar - frame at the top of the stem, box pushed up by its own half
-               thickness so it rests ON the stem rather than straddling the
-               top face.
-  Every link needs a non-zero <inertial> or Gazebo silently drops it, even
-  though both of these are static.
+    stem      - frame at ground level, box pushed up by stem_height/2 so it
+                stands ON the ground instead of being half buried. Its top
+                face therefore lands at exactly z = stem_height.
+    crossbar  - frame at the top of the stem, box pushed up by its own half
+                thickness so it rests ON the stem rather than straddling the
+                top face.
+    upper_arm - frame at the shoulder pivot, box pushed DOWN by half its
+                length so it hangs below the joint.
+  "Right" is -Y, following the usual robotics convention of +X forward,
+  +Y left, +Z up.
+  The shoulder joint is deliberately passive: no controller, no PID, just
+  damping and friction. The arm falls under gravity and swings like a real
+  pendulum, which is the point of the rig.
+  Every link needs a non-zero <inertial> or Gazebo silently drops it.
   Build standalone:
     xacro urdf/rig.urdf.xacro > rig.urdf
@@ -36,4 +43,15 @@
   <xacro:property name="cd" value="$(arg crossbar_depth)"/>
   <xacro:property name="crossbar_mass" value="4.0"/>
+  <!-- upper arm: hangs from the right end of the crossbar.
+       Half the stem length, per the build spec. -->
+  <xacro:arg name="upper_arm_width" default="0.07"/>
+  <xacro:arg name="upper_arm_depth" default="0.07"/>
+  <xacro:property name="ual" value="${sh/2.0}"/>
+  <xacro:property name="uaw" value="$(arg upper_arm_width)"/>
+  <xacro:property name="uad" value="$(arg upper_arm_depth)"/>
+  <xacro:property name="upper_arm_mass" value="2.0"/>
+  <!-- passive shoulder: damping/friction only, no actuator -->
+  <xacro:property name="shoulder_damping"  value="0.2"/>
+  <xacro:property name="shoulder_friction" value="0.1"/>
   <material name="grey">
     <color rgba="0.4 0.4 0.45 1.0"/>
@@ -41,4 +59,7 @@
   <material name="steel_blue">
     <color rgba="0.25 0.35 0.5 1.0"/>
+  </material>
+  <material name="copper">
+    <color rgba="0.72 0.45 0.20 1.0"/>
   </material>
   <!-- ================= links ================= -->
@@ -97,4 +118,30 @@
     </inertial>
   </link>
+  <!-- upper arm.
+       Frame is at the shoulder pivot; geometry hangs DOWN from it, hence the
+       negative z offset. Length is half the stem height. -->
+  <link name="upper_arm">
+    <visual>
+      <origin xyz="0 0 ${-ual/2}" rpy="0 0 0"/>
+      <geometry>
+        <box size="${uad} ${uaw} ${ual}"/>
+      </geometry>
+      <material name="copper"/>
+    </visual>
+    <collision>
+      <origin xyz="0 0 ${-ual/2}" rpy="0 0 0"/>
+      <geometry>
+        <box size="${uad} ${uaw} ${ual}"/>
+      </geometry>
+    </collision>
+    <inertial>
+      <origin xyz="0 0 ${-ual/2}" rpy="0 0 0"/>
+      <mass value="${upper_arm_mass}"/>
+      <inertia
+        ixx="${upper_arm_mass*(uaw*uaw + ual*ual)/12.0}" ixy="0.0" ixz="0.0"
+        iyy="${upper_arm_mass*(uad*uad + ual*ual)/12.0}" iyz="0.0"
+        izz="${upper_arm_mass*(uad*uad + uaw*uaw)/12.0}"/>
+    </inertial>
+  </link>
   <!-- ================= joints ================= -->
   <joint name="world_to_stem" type="fixed">
@@ -109,15 +156,20 @@
     <origin xyz="0 0 ${sh}" rpy="0 0 0"/>
   </joint>
+  <!-- Shoulder. Sits at the RIGHT end of the crossbar (-Y) and level with
+       the crossbar's own frame, i.e. the underside of the bar.
+       Rotation is about X, so the arm swings in the Y-Z plane - the same
+       plane the crossbar lies in. Passive: no transmission, no controller,
+       so it simply falls and swings under gravity. -->
+  <joint name="shoulder_joint" type="revolute">
+    <parent link="crossbar"/>
+    <child  link="upper_arm"/>
+    <origin xyz="0 ${-cl/2} 0" rpy="0 0 0"/>
+    <axis   xyz="1 0 0"/>
+    <limit lower="${-pi}" upper="${pi}" effort="100.0" velocity="5.0"/>
+    <dynamics damping="${shoulder_damping}" friction="${shoulder_friction}"/>
+  </joint>
   <!--
-    STAGE 3 goes here - an arm hanging off one end of the crossbar. Swap
-    fixed for revolute and give it an axis, limits and dynamics, e.g.
-      <joint name="crossbar_to_upper_arm" type="revolute">
-        <parent link="crossbar"/>
-        <child  link="upper_arm"/>
-        <origin xyz="0 ${cl/2} 0" rpy="0 0 0"/>
-        <axis   xyz="0 1 0"/>
-        <limit lower="-3.14" upper="3.14" effort="100" velocity="5"/>
-        <dynamics damping="0.2" friction="0.1"/>
-      </joint>
+    STAGE 4 goes here - forearm on an elbow joint, hanging off the bottom
+    of the upper arm at xyz="0 0 ${-ual}".
   -->
   <!-- ================= gazebo ================= -->
@@ -132,4 +184,9 @@
     <mu2>0.8</mu2>
   </gazebo>
+  <gazebo reference="upper_arm">
+    <material>Gazebo/Orange</material>
+    <mu1>0.8</mu1>
+    <mu2>0.8</mu2>
+  </gazebo>
   <!-- Exposes /gazebo/get_link_state, /gazebo/apply_body_wrench, etc. so the
        rig can be poked from the command line later. -->

Commit message: arm-rig: mount arm outboard on the +Y end of the crossbar
Was centred on the -Y end and hanging from the bar's underside. Now:

- pivot moved to +Y (arm_side arg, default 1, flip with --arm-side -1)
- offset half an arm-width past the bar end so the crossbar's end face
  sits flush against the arm's inner side face, no overlap
- raised by crossbar_thickness so the arm's top face is level with the
  top of the crossbar rather than its underside

File: projects/3d/gazebo/URDF-Humanoid-Arm/urdf/rig.urdf.xacro (robot description, xacro)
@@ -16,6 +16,9 @@
     upper_arm - frame at the shoulder pivot, box pushed DOWN by half its
                 length so it hangs below the joint.
-  "Right" is -Y, following the usual robotics convention of +X forward,
-  +Y left, +Z up.
+  The arm hangs OUTBOARD of the crossbar, not underneath it: the end face of
+  the crossbar meets the inner side face of the arm, and the top face of the
+  arm is level with the top face of the crossbar. Hence the pivot is offset
+  by half the arm width past the crossbar end.
+  arm_side flips which end it hangs from: +1 or -1 along Y.
   The shoulder joint is deliberately passive: no controller, no PID, just
   damping and friction. The arm falls under gravity and swings like a real
@@ -51,4 +54,10 @@
   <xacro:property name="uad" value="$(arg upper_arm_depth)"/>
   <xacro:property name="upper_arm_mass" value="2.0"/>
+  <!-- which end of the crossbar the arm hangs from: +1 or -1 along Y -->
+  <xacro:arg name="arm_side" default="1"/>
+  <xacro:property name="side" value="$(arg arm_side)"/>
+  <!-- Pivot sits half an arm-width PAST the crossbar end, so the crossbar's
+       end face lands flush against the arm's inner side face. -->
+  <xacro:property name="shoulder_y" value="${side*(cl/2.0 + uaw/2.0)}"/>
   <!-- passive shoulder: damping/friction only, no actuator -->
   <xacro:property name="shoulder_damping"  value="0.2"/>
@@ -156,6 +165,6 @@
     <origin xyz="0 0 ${sh}" rpy="0 0 0"/>
   </joint>
-  <!-- Shoulder. Sits at the RIGHT end of the crossbar (-Y) and level with
-       the crossbar's own frame, i.e. the underside of the bar.
+  <!-- Shoulder. Sits just past the end of the crossbar so the bar's end face
+       butts against the arm's inner side face, with the two top faces level.
        Rotation is about X, so the arm swings in the Y-Z plane - the same
        plane the crossbar lies in. Passive: no transmission, no controller,
@@ -164,5 +173,5 @@
     <parent link="crossbar"/>
     <child  link="upper_arm"/>
-    <origin xyz="0 ${-cl/2} 0" rpy="0 0 0"/>
+    <origin xyz="0 ${shoulder_y} ${ct}" rpy="0 0 0"/>
     <axis   xyz="1 0 0"/>
     <limit lower="${-pi}" upper="${pi}" effort="100.0" velocity="5.0"/>

Commit message: arm-rig: slider GUI for the shoulder angle
- shoulder_joint revolute -> continuous, so it can be driven a full
  0-360 and wrap instead of stopping at +/-pi
- arm_gui.py: single 0-360 slider, re-asserts the target through
  /gazebo/set_model_configuration at 30 Hz so the pose holds against
  gravity (the joint is still passive, nothing actuates it)
- Release button drops the hold and lets the arm swing; the slider then
  follows the real joint angle instead of driving it
- 2-arm-gui.sh wrapper to source ROS the same way the launcher does

File: projects/3d/gazebo/URDF-Humanoid-Arm/urdf/rig.urdf.xacro (robot description, xacro)
@@ -168,12 +168,14 @@
        butts against the arm's inner side face, with the two top faces level.
        Rotation is about X, so the arm swings in the Y-Z plane - the same
-       plane the crossbar lies in. Passive: no transmission, no controller,
-       so it simply falls and swings under gravity. -->
-  <joint name="shoulder_joint" type="revolute">
+       plane the crossbar lies in.
+       "continuous" rather than "revolute": no limits, so the arm can be
+       driven through a full 0-360 and wrap round. Still passive - no
+       transmission and no controller - so left alone it just falls and
+       swings under gravity. arm_gui.py drives it kinematically. -->
+  <joint name="shoulder_joint" type="continuous">
     <parent link="crossbar"/>
     <child  link="upper_arm"/>
     <origin xyz="0 ${shoulder_y} ${ct}" rpy="0 0 0"/>
     <axis   xyz="1 0 0"/>
-    <limit lower="${-pi}" upper="${pi}" effort="100.0" velocity="5.0"/>
     <dynamics damping="${shoulder_damping}" friction="${shoulder_friction}"/>
   </joint>

Commit message: arm-rig: swing the shoulder about Y (green) instead of X (red)
Arm now sweeps forward/back in the X-Z plane. The pivot axis runs along
the crossbar's own long axis, so the arm sweeps clear of the bar rather
than through the plane it occupies.

File: projects/3d/gazebo/URDF-Humanoid-Arm/urdf/rig.urdf.xacro (robot description, xacro)
@@ -20,4 +20,6 @@
   arm is level with the top face of the crossbar. Hence the pivot is offset
   by half the arm width past the crossbar end.
+  The shoulder rotates about Y - the green axis in Gazebo - so the arm
+  swings forward/back in the X-Z plane.
   arm_side flips which end it hangs from: +1 or -1 along Y.
   The shoulder joint is deliberately passive: no controller, no PID, just
@@ -167,6 +169,8 @@
   <!-- Shoulder. Sits just past the end of the crossbar so the bar's end face
        butts against the arm's inner side face, with the two top faces level.
-       Rotation is about X, so the arm swings in the Y-Z plane - the same
-       plane the crossbar lies in.
+       Rotation is about Y (the GREEN axis), so the arm swings forward and
+       back in the X-Z plane - perpendicular to the crossbar. Because the
+       pivot axis runs along the crossbar's own long axis, the arm sweeps
+       clear of the bar instead of into it.
        "continuous" rather than "revolute": no limits, so the arm can be
        driven through a full 0-360 and wrap round. Still passive - no
@@ -177,5 +181,5 @@
     <child  link="upper_arm"/>
     <origin xyz="0 ${shoulder_y} ${ct}" rpy="0 0 0"/>
-    <axis   xyz="1 0 0"/>
+    <axis   xyz="0 1 0"/>
     <dynamics damping="${shoulder_damping}" friction="${shoulder_friction}"/>
   </joint>

Commit message: arm-rig: pivot on the crossbar end-face centre, arm hung from its top edge
Previously the pivot sat half an arm-width past the bar end and level
with the bar's top face, so the arm's top corners swept up above the
crossbar as soon as it rotated.

Now the pivot is at the centre of the crossbar's end face (on the end,
halfway up), and that point is the arm's top inner edge rather than its
top-face centre. The arm top therefore sits 0.04 m below the bar top and
the swept corners stay under it - guaranteed while
upper_arm_depth <= crossbar_thickness.

File: projects/3d/gazebo/URDF-Humanoid-Arm/urdf/rig.urdf.xacro (robot description, xacro)
@@ -14,10 +14,13 @@
                 thickness so it rests ON the stem rather than straddling the
                 top face.
-    upper_arm - frame at the shoulder pivot, box pushed DOWN by half its
-                length so it hangs below the joint.
-  The arm hangs OUTBOARD of the crossbar, not underneath it: the end face of
-  the crossbar meets the inner side face of the arm, and the top face of the
-  arm is level with the top face of the crossbar. Hence the pivot is offset
-  by half the arm width past the crossbar end.
+    upper_arm - frame at the shoulder pivot, box hung DOWN and OUTBOARD of
+                it, so the pivot lands on the arm's top inner edge.
+  Where the two meet: the pivot sits at the centre of the crossbar's end
+  face - halfway up it, right on the end - and that same point is the arm's
+  top inner edge. So the arm's top face is half a crossbar-thickness BELOW
+  the top of the bar and cannot poke up through it.
+  That clearance holds while swinging too, as long as
+  upper_arm_depth <= crossbar_thickness: the top corners sweep a radius of
+  upper_arm_depth/2 about the pivot, which stays inside the bar's top face.
   The shoulder rotates about Y - the green axis in Gazebo - so the arm
   swings forward/back in the X-Z plane.
@@ -59,7 +62,7 @@
   <xacro:arg name="arm_side" default="1"/>
   <xacro:property name="side" value="$(arg arm_side)"/>
-  <!-- Pivot sits half an arm-width PAST the crossbar end, so the crossbar's
-       end face lands flush against the arm's inner side face. -->
-  <xacro:property name="shoulder_y" value="${side*(cl/2.0 + uaw/2.0)}"/>
+  <!-- Pivot sits ON the crossbar's end face, halfway up it. -->
+  <xacro:property name="shoulder_y" value="${side*cl/2.0}"/>
+  <xacro:property name="shoulder_z" value="${ct/2.0}"/>
   <!-- passive shoulder: damping/friction only, no actuator -->
   <xacro:property name="shoulder_damping"  value="0.2"/>
@@ -130,9 +133,10 @@
   </link>
   <!-- upper arm.
-       Frame is at the shoulder pivot; geometry hangs DOWN from it, hence the
-       negative z offset. Length is half the stem height. -->
+       Frame is at the shoulder pivot, which sits on the arm's top INNER
+       edge - hence the geometry is offset both down (-z) and outboard
+       (+/-y) from it. Length is half the stem height. -->
   <link name="upper_arm">
     <visual>
-      <origin xyz="0 0 ${-ual/2}" rpy="0 0 0"/>
+      <origin xyz="0 ${side*uaw/2} ${-ual/2}" rpy="0 0 0"/>
       <geometry>
         <box size="${uad} ${uaw} ${ual}"/>
@@ -141,5 +145,5 @@
     </visual>
     <collision>
-      <origin xyz="0 0 ${-ual/2}" rpy="0 0 0"/>
+      <origin xyz="0 ${side*uaw/2} ${-ual/2}" rpy="0 0 0"/>
       <geometry>
         <box size="${uad} ${uaw} ${ual}"/>
@@ -147,5 +151,5 @@
     </collision>
     <inertial>
-      <origin xyz="0 0 ${-ual/2}" rpy="0 0 0"/>
+      <origin xyz="0 ${side*uaw/2} ${-ual/2}" rpy="0 0 0"/>
       <mass value="${upper_arm_mass}"/>
       <inertia
@@ -167,6 +171,8 @@
     <origin xyz="0 0 ${sh}" rpy="0 0 0"/>
   </joint>
-  <!-- Shoulder. Sits just past the end of the crossbar so the bar's end face
-       butts against the arm's inner side face, with the two top faces level.
+  <!-- Shoulder. Pivot is at the centre of the crossbar's end face: right on
+       the end, halfway up the bar. That same point is the arm's top inner
+       edge, so the arm hangs just below the bar's top surface instead of
+       being level with it.
        Rotation is about Y (the GREEN axis), so the arm swings forward and
        back in the X-Z plane - perpendicular to the crossbar. Because the
@@ -180,5 +186,5 @@
     <parent link="crossbar"/>
     <child  link="upper_arm"/>
-    <origin xyz="0 ${shoulder_y} ${ct}" rpy="0 0 0"/>
+    <origin xyz="0 ${shoulder_y} ${shoulder_z}" rpy="0 0 0"/>
     <axis   xyz="0 1 0"/>
     <dynamics damping="${shoulder_damping}" friction="${shoulder_friction}"/>

Commit message: arm-rig: raise the arm so its top is level with the crossbar top
The pivot sits at the bar's mid-height, and the arm was hung with its top
face AT the pivot, leaving a 0.04 m step below the bar's top surface.
Geometry is now offset up by ct/2 so the arm covers the full height of
the end face.

Pivot is still ct/2 below the arm's top, so the corners rise at most
0.013 m above the bar top mid-swing (peaks around 45 deg) rather than the
0.035 m they would if the pivot were on the top face.

File: projects/3d/gazebo/URDF-Humanoid-Arm/urdf/rig.urdf.xacro (robot description, xacro)
@@ -14,13 +14,13 @@
                 thickness so it rests ON the stem rather than straddling the
                 top face.
-    upper_arm - frame at the shoulder pivot, box hung DOWN and OUTBOARD of
-                it, so the pivot lands on the arm's top inner edge.
+    upper_arm - box hung DOWN and OUTBOARD of the shoulder pivot, raised so
+                its top face is level with the top of the crossbar.
   Where the two meet: the pivot sits at the centre of the crossbar's end
-  face - halfway up it, right on the end - and that same point is the arm's
-  top inner edge. So the arm's top face is half a crossbar-thickness BELOW
-  the top of the bar and cannot poke up through it.
-  That clearance holds while swinging too, as long as
-  upper_arm_depth <= crossbar_thickness: the top corners sweep a radius of
-  upper_arm_depth/2 about the pivot, which stays inside the bar's top face.
+  face - halfway up it, right on the end. The arm's inner face is flush
+  against that end face and its top face is level with the bar's top, so the
+  arm covers the full height of the end face with no step.
+  The pivot is therefore NOT at the arm's top face but half a crossbar
+  thickness below it, which is what stops the arm lifting clear of the bar
+  when it swings.
   The shoulder rotates about Y - the green axis in Gazebo - so the arm
   swings forward/back in the X-Z plane.
@@ -133,10 +133,10 @@
   </link>
   <!-- upper arm.
-       Frame is at the shoulder pivot, which sits on the arm's top INNER
-       edge - hence the geometry is offset both down (-z) and outboard
-       (+/-y) from it. Length is half the stem height. -->
+       Geometry sits outboard of the pivot in Y and is raised by ct/2 in Z so
+       its top face is level with the top of the crossbar rather than with
+       the pivot itself. Length is half the stem height. -->
   <link name="upper_arm">
     <visual>
-      <origin xyz="0 ${side*uaw/2} ${-ual/2}" rpy="0 0 0"/>
+      <origin xyz="0 ${side*uaw/2} ${ct/2 - ual/2}" rpy="0 0 0"/>
       <geometry>
         <box size="${uad} ${uaw} ${ual}"/>
@@ -145,5 +145,5 @@
     </visual>
     <collision>
-      <origin xyz="0 ${side*uaw/2} ${-ual/2}" rpy="0 0 0"/>
+      <origin xyz="0 ${side*uaw/2} ${ct/2 - ual/2}" rpy="0 0 0"/>
       <geometry>
         <box size="${uad} ${uaw} ${ual}"/>
@@ -151,5 +151,5 @@
     </collision>
     <inertial>
-      <origin xyz="0 ${side*uaw/2} ${-ual/2}" rpy="0 0 0"/>
+      <origin xyz="0 ${side*uaw/2} ${ct/2 - ual/2}" rpy="0 0 0"/>
       <mass value="${upper_arm_mass}"/>
       <inertia
@@ -172,7 +172,7 @@
   </joint>
   <!-- Shoulder. Pivot is at the centre of the crossbar's end face: right on
-       the end, halfway up the bar. That same point is the arm's top inner
-       edge, so the arm hangs just below the bar's top surface instead of
-       being level with it.
+       the end, halfway up the bar. The arm's inner face is flush against
+       that end face and its top is level with the bar's top, so the pivot
+       sits just inside the arm near its top inner edge.
        Rotation is about Y (the GREEN axis), so the arm swings forward and
        back in the X-Z plane - perpendicular to the crossbar. Because the
